File: Statemachine/brd/Statemachine_ST7735.sch (EAGLE design)
At the start: 11 parts

Commit message: add sd card
Connections:
- removed net MOSI: JP3.10
- removed net SCLK: JP3.9
- net CS-SD: now also U$1.D4
- net MISO: now also U$1.D12
- net SCL: now also JP3.9
- net SDA: now also JP3.10
Other:
- note added: "MISO"
- note added: "MOSI"
- note added: "SCLK"
- moved on the sheet: JP1, JP3, JP4, R3, R4
