File: Statemachine/brd/Statemachine_ST7735.R03.brd (EAGLE design)
At the start: 100 x 76.2 mm, 18 parts

Commit message: add board
Routing:
- net GND: track 0.00 -> 293.2 mm, vias 0 -> 6
- net LCD-RES: track 46.6 -> 39.7 mm
- net +5V: track 226.7 -> 231.7 mm
- net BTN2: track 132.9 -> 132.2 mm
- removed copper zone on layer 16, net GND
Changed lines of the file:
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@@
 <setting verticaltext="up"/>
 </settings>
-<grid distance="0.05" unitdist="inch" unit="inch" style="lines" multiple="1" display="yes" altdistance="0.05" altunitdist="inch" altunit="inch"/>
+<grid distance="0.1" unitdist="inch" unit="inch" style="lines" multiple="1" display="yes" altdistance="0.05" altunitdist="inch" altunit="inch"/>
 <layers>
 <layer number="1" name="Top" color="4" fill="1" visible="yes" active="yes"/>
@@
 <layer number="25" name="tNames" color="7" fill="1" visible="yes" active="yes"/>
 <layer number="26" name="bNames" color="7" fill="1" visible="yes" active="yes"/>
-<layer number="27" name="tValues" color="7" fill="1" visible="no" active="yes"/>
-<layer number="28" name="bValues" color="7" fill="1" visible="no" active="yes"/>
+<layer number="27" name="tValues" color="7" fill="1" visible="yes" active="yes"/>
+<layer number="28" name="bValues" color="7" fill="1" visible="yes" active="yes"/>
 <layer number="29" name="tStop" color="7" fill="3" visible="no" active="yes"/>
 <layer number="30" name="bStop" color="7" fill="6" visible="no" active="yes"/>
@@
 <wire x1="11.43" y1="55.88" x2="25.4" y2="55.88" width="0.4064" layer="16"/>
 <wire x1="25.4" y1="55.88" x2="25.4" y2="60.96" width="0.4064" layer="16"/>
-<wire x1="25.4" y1="55.88" x2="25.4" y2="66.04" width="0.4064" layer="16"/>
-<wire x1="25.4" y1="66.04" x2="26.67" y2="67.31" width="0.4064" layer="16"/>
-<wire x1="26.67" y1="67.31" x2="87.63" y2="67.31" width="0.4064" layer="16"/>
-<wire x1="87.63" y1="67.31" x2="88.9" y2="66.04" width="0.4064" layer="16"/>
-<wire x1="88.9" y1="66.04" x2="88.9" y2="60.96" width="0.4064" layer="16"/>
+<wire x1="25.4" y1="55.88" x2="25.4" y2="68.58" width="0.4064" layer="16"/>
+<wire x1="25.4" y1="68.58" x2="26.67" y2="69.85" width="0.4064" layer="16"/>
+<wire x1="26.67" y1="69.85" x2="87.63" y2="69.85" width="0.4064" layer="16"/>
+<wire x1="87.63" y1="69.85" x2="88.9" y2="68.58" width="0.4064" layer="16"/>
+<wire x1="88.9" y1="68.58" x2="88.9" y2="60.96" width="0.4064" layer="16"/>
 <wire x1="77.47" y1="48.26" x2="88.9" y2="48.26" width="0.4064" layer="16"/>
 <wire x1="88.9" y1="17.78" x2="92.71" y2="17.78" width="0.4064" layer="16"/>
@@
 <wire x1="92.71" y1="34.29" x2="93.98" y2="35.56" width="0.4064" layer="16"/>
 <wire x1="69.85" y1="50.8" x2="69.85" y2="48.26" width="0.4064" layer="16"/>
-<wire x1="67.31" y1="48.26" x2="77.47" y2="48.26" width="0.4064" layer="16"/>
-<wire x1="69.85" y1="48.26" x2="72.39" y2="48.26" width="0" layer="19" extent="1-1"/>
-<wire x1="67.31" y1="48.26" x2="69.85" y2="48.26" width="0" layer="19" extent="1-1"/>
+<wire x1="72.39" y1="48.26" x2="77.47" y2="48.26" width="0.4064" layer="16"/>
+<wire x1="69.85" y1="48.26" x2="72.39" y2="48.26" width="0.4064" layer="16"/>
+<wire x1="69.85" y1="48.26" x2="67.31" y2="48.26" width="0.4064" layer="16"/>
 </signal>
 <signal name="GND">
@@
 <contactref element="S3" pad="3"/>
 <contactref element="S1" pad="3"/>
-<polygon width="0.4064" layer="16" spacing="32.258" isolate="0.3048">
-<vertex x="0" y="76.2"/>
-<vertex x="100.33" y="76.2"/>
-<vertex x="100.33" y="0"/>
-<vertex x="0" y="0"/>
-</polygon>
 <contactref element="JP5" pad="4"/>
+<wire x1="7.62" y1="27.94" x2="6.35" y2="27.94" width="0.4064" layer="16"/>
+<wire x1="6.35" y1="27.94" x2="5.08" y2="29.21" width="0.4064" layer="16"/>
+<wire x1="5.08" y1="29.21" x2="5.08" y2="52.07" width="0.4064" layer="16"/>
+<wire x1="5.08" y1="52.07" x2="6.35" y2="53.34" width="0.4064" layer="16"/>
+<wire x1="6.35" y1="53.34" x2="7.62" y2="53.34" width="0.4064" layer="16"/>
+<wire x1="88.9" y1="58.42" x2="90.17" y2="58.42" width="0.4064" layer="16"/>
+<wire x1="90.17" y1="58.42" x2="91.44" y2="57.15" width="0.4064" layer="16"/>
+<wire x1="91.44" y1="57.15" x2="91.44" y2="50.8" width="0.4064" layer="16"/>
+<via x="91.44" y="50.8" extent="1-16" drill="0.6" shape="square"/>
+<wire x1="91.44" y1="50.8" x2="91.44" y2="45.72" width="0.4064" layer="1"/>
+<via x="91.44" y="45.72" extent="1-16" drill="0.6" shape="square"/>
+<wire x1="91.44" y1="45.72" x2="91.44" y2="41.91" width="0.4064" layer="16"/>
+<wire x1="91.44" y1="41.91" x2="90.17" y2="40.64" width="0.4064" layer="16"/>
+<wire x1="88.9" y1="40.64" x2="90.17" y2="40.64" width="0.4064" layer="16"/>
+<wire x1="90.17" y1="40.64" x2="91.44" y2="39.37" width="0.4064" layer="16"/>
+<wire x1="91.44" y1="39.37" x2="91.44" y2="35.56" width="0.4064" layer="16"/>
+<via x="91.44" y="35.56" extent="1-16" drill="0.6" shape="square"/>
+<wire x1="91.44" y1="35.56" x2="91.44" y2="30.48" width="0.4064" layer="1"/>
+<via x="91.44" y="30.48" extent="1-16" drill="0.6" shape="square"/>
+<wire x1="91.44" y1="30.48" x2="91.44" y2="26.67" width="0.4064" layer="16"/>
+<wire x1="91.44" y1="26.67" x2="90.17" y2="25.4" width="0.4064" layer="16"/>
+<wire x1="90.17" y1="25.4" x2="88.9" y2="25.4" width="0.4064" layer="16"/>
+<wire x1="88.9" y1="25.4" x2="87.63" y2="25.4" width="0.4064" layer="16"/>
+<wire x1="87.63" y1="25.4" x2="86.36" y2="24.13" width="0.4064" layer="16"/>
+<wire x1="86.36" y1="24.13" x2="86.36" y2="16.51" width="0.4064" layer="16"/>
+<wire x1="86.36" y1="16.51" x2="87.63" y2="15.24" width="0.4064" layer="16"/>
+<wire x1="27.94" y1="60.96" x2="27.94" y2="58.42" width="0.4064" layer="16"/>
+<via x="27.94" y="58.42" extent="1-16" drill="0.6" shape="square"/>
+<wire x1="27.94" y1="58.42" x2="22.86" y2="58.42" width="0.4064" layer="1"/>
+<via x="22.86" y="58.42" extent="1-16" drill="0.6" shape="square"/>
+<wire x1="22.86" y1="58.42" x2="8.89" y2="58.42" width="0.4064" layer="16"/>
+<wire x1="8.89" y1="58.42" x2="7.62" y2="57.15" width="0.4064" layer="16"/>
+<wire x1="7.62" y1="57.15" x2="7.62" y2="53.34" width="0.4064" layer="16"/>
+<wire x1="27.94" y1="58.42" x2="27.94" y2="66.04" width="0.4064" layer="16"/>
+<wire x1="27.94" y1="66.04" x2="29.21" y2="67.31" width="0.4064" layer="16"/>
+<wire x1="29.21" y1="67.31" x2="63.5" y2="67.31" width="0.4064" layer="16"/>
+<wire x1="63.5" y1="67.31" x2="64.77" y2="66.04" width="0.4064" layer="16"/>
+<wire x1="64.77" y1="66.04" x2="64.77" y2="50.8" width="0.4064" layer="16"/>
+<wire x1="64.77" y1="50.8" x2="62.23" y2="48.26" width="0.4064" layer="16"/>
+<wire x1="88.9" y1="15.24" x2="87.63" y2="15.24" width="0.4064" layer="16"/>
+<wire x1="87.63" y1="15.24" x2="86.36" y2="13.97" width="0.4064" layer="16"/>
+<wire x1="86.36" y1="13.97" x2="86.36" y2="2.54" width="0.4064" layer="16"/>
+<wire x1="86.36" y1="2.54" x2="85.09" y2="1.27" width="0.4064" layer="16"/>
+<wire x1="85.09" y1="1.27" x2="25.4" y2="1.27" width="0.4064" layer="16"/>
+<wire x1="25.4" y1="1.27" x2="22.86" y2="3.81" width="0.4064" layer="16"/>
+<wire x1="22.86" y1="3.81" x2="22.86" y2="17.78" width="0.4064" layer="16"/>
+<wire x1="22.86" y1="17.78" x2="21.59" y2="19.05" width="0.4064" layer="16"/>
+<wire x1="21.59" y1="19.05" x2="6.35" y2="19.05" width="0.4064" layer="16"/>
+<wire x1="6.35" y1="19.05" x2="5.08" y2="20.32" width="0.4064" layer="16"/>
+<wire x1="5.08" y1="20.32" x2="5.08" y2="29.21" width="0.4064" layer="16"/>
 </signal>
 <signal name="BTN1">
@@
 <wire x1="80.01" y1="27.94" x2="81.28" y2="26.67" width="0.4064" layer="16"/>
 <wire x1="29.21" y1="6.35" x2="27.94" y2="7.62" width="0.4064" layer="16"/>
-<wire x1="27.94" y1="7.62" x2="27.94" y2="46.99" width="0.4064" layer="16"/>
-<wire x1="27.94" y1="46.99" x2="26.67" y2="48.26" width="0.4064" layer="16"/>
-<wire x1="26.67" y1="48.26" x2="25.4" y2="48.26" width="0.4064" layer="16"/>
+<wire x1="27.94" y1="7.62" x2="27.94" y2="35.56" width="0.4064" layer="16"/>
+<wire x1="27.94" y1="35.56" x2="25.4" y2="38.1" width="0.4064" layer="16"/>
+<wire x1="25.4" y1="38.1" x2="25.4" y2="48.26" width="0.4064" layer="16"/>
 <wire x1="29.21" y1="6.35" x2="80.01" y2="6.35" width="0.4064" layer="16"/>
 <wire x1="80.01" y1="6.35" x2="81.28" y2="7.62" width="0.4064" layer="16"/>
@@
 <contactref element="JP3" pad="6"/>
 <contactref element="NANO" pad="RESET"/>
-<wire x1="62.23" y1="50.8" x2="63.5" y2="50.8" width="0.4064" layer="16"/>
-<wire x1="63.5" y1="50.8" x2="66.04" y2="53.34" width="0.4064" layer="16"/>
-<wire x1="66.04" y1="53.34" x2="66.04" y2="63.5" width="0.4064" layer="16"/>
-<wire x1="66.04" y1="63.5" x2="64.77" y2="64.77" width="0.4064" layer="16"/>
-<wire x1="64.77" y1="64.77" x2="39.37" y2="64.77" width="0.4064" layer="16"/>
+<wire x1="62.23" y1="50.8" x2="58.42" y2="50.8" width="0.4064" layer="16"/>
+<wire x1="58.42" y1="50.8" x2="57.15" y2="52.07" width="0.4064" layer="16"/>
+<wire x1="57.15" y1="52.07" x2="57.15" y2="63.5" width="0.4064" layer="16"/>
+<wire x1="57.15" y1="63.5" x2="55.88" y2="64.77" width="0.4064" layer="16"/>
+<wire x1="55.88" y1="64.77" x2="39.37" y2="64.77" width="0.4064" layer="16"/>
 <wire x1="39.37" y1="64.77" x2="38.1" y2="63.5" width="0.4064" layer="16"/>
 <wire x1="38.1" y1="63.5" x2="38.1" y2="60.96" width="0.4064" layer="16"/>
