File: Statemachine_ST7783_ADC/PCB/rtc-shield.sch (EAGLE design)
At the start: 56 parts, among them IC1 TLC2543, IC2 RV_3049_C2, J10 MC1,5/2-G-3,5, J11 MC1,5/2-G-3,5, J12 MC1,5/2-G-3,5, J13 MC1,5/2-G-3,5, J14 MC1,5/2-G-3,5, J15 MC1,5/2-G-3,5, J16 MC1,5/2-G-3,5, J9 MC1,5/2-G-3,5

Commit message: PCB: add reset note MainScreen: change gauges, try to optimize redrawing.
Parts:
- removed AD: 6x1F-H8.5, SmartPrj:PINHD-1X6
- removed C10, C11, C12, C13, C19, C2, C20, C21, C22, C23, C24, C25, C26, C5, C8, C9: 10n, Passiv:C_KER
- removed C16, C3, C6: 100n, Passiv:C_KER
- removed IC1: TLC2543, HL_IC1:TLC2543
- removed IOH: 10x1F-H8.5, SmartPrj:PINHD-1X10_ARD
- removed IOL, POWER: 8x1F-H8.5, SmartPrj:PINHD-1X8
- removed J10, J11, J12, J13, J14, J15, J16, J9: MC1,5/2-G-3,5, PHOENIX:MC1,5/2-G-3,5
- removed R10, R13, R14, R15, R16, R17, R6, R7, R8, R9: 2K, Passiv:R@2
- removed R11, R12, R18, R19, R2, R20, R21, R3: 10K, Passiv:R@2
- removed R4: 1K21, Passiv:R@2
- removed R5: 909R, Passiv:R@2
- added JP1: (no value), arduino_adafruit:PINHD-1X6B
- added JP3, JP4: (no value), arduino_adafruit:PINHD-1X1CB
Connections:
- removed net +3V3: POWER.4
- removed net AD0: AD.1
- removed net AD1: AD.2
- removed net AD2: AD.3
- removed net AD3: AD.4
- removed net AD4/SDA: AD.5, IC1./CS, IOH.9
- removed net AD5/SCL: AD.6, IOH.10
- removed net AREF: IOH.8
- removed net IO0: IOL.1
- removed net IO1: IOL.2
- removed net IO2: IOL.3
- removed net IO3: IOL.4
- removed net IO4: IOL.5
- removed net IO5: IOL.6
- removed net IO6: IOL.7
- removed net IO7: IOL.8
- removed net IO8: IOH.1
- removed net IO9: IOH.2
- removed net N$10: C3.2, IC1.REF-, R5.1, R6.2
- removed net N$11: C6.2, IC1.REF+, R4.1, R7.2
- removed net N$16: C2.2, IC1.AIN1, R11.2
- removed net N$17: C8.2, IC1.AIN2, R2.2
- removed net N$18: C9.2, IC1.AIN3, R3.2
- removed net N$19: C5.2, IC1.AIN0, R12.2
- removed net N$20: C23.2, IC1.AIN4, R18.2
- removed net N$21: C24.2, IC1.AIN5, R19.2
- removed net N$22: C25.2, IC1.AIN6, R20.2
- removed net N$23: C26.2, IC1.AIN7, R21.2
- removed net SS: IOH.3
- removed net VIN: POWER.8
- removed net X1_RX4-: C13.2, J9.1.1, R12.1, R9.1
- removed net X2_TX4-: C12.2, J10.1.1, R11.1, R13.1
- removed net X3_RX3-: C10.2, J11.1.1, R10.1, R2.1
- removed net X4_TX3-: C11.2, J12.1.1, R3.1, R8.1
- removed net X5_RX2-: C19.2, J13.1.1, R14.1, R18.1
- removed net X6_TX2-: C21.2, J14.1.1, R15.1, R19.1
- removed net X7_RX1-: C20.2, J15.1.1, R16.1, R20.1
- removed net X8_TX1-: C22.2, J16.1.1, R17.1, R21.1
- new net N$1: IC2.CLKOE, JP3.1
- new net N$2: IC2.!INT, JP4.1
- net +5V: now also JP1.1; no longer C16.2, IC1.VCC, POWER.2, POWER.5, R10.2, R13.2, R14.2, R15.2, R16.2, R17.2, R6.1, R7.1, R8.2, R9.2
- net GND: now also JP1.6; no longer C10.1, C11.1, C12.1, C13.1, C16.1, C19.1, C2.1, C20.1, C21.1, C22.1, C23.1, C24.1, C25.1, C26.1, C3.1, C5.1, C6.1, C8.1, C9.1, IC1.GND, IOH.7, J10.2.1, J11.2.1, J12.2.1, J13.2.1, J14.2.1, J15.2.1, J16.2.1, J9.2.1, POWER.6, POWER.7, R4.2, R5.2
- net MISO: no longer IC1.DATOUT, IOH.5
- net MOSI: no longer IC1.DATIN, IOH.4
- net SCK: no longer IC1.CLK, IOH.6
Other:
- note added: "RTC Shield"
- note removed: "0"
- note removed: "1"
- note removed: "10"
- note removed: "11"
- note removed: "12"
- note removed: "13"
- note removed: "2"
- note removed: "3"
- note removed: "4"
- note removed: "5"
- note removed: "6"
- note removed: "7"
- note removed: "8"
- note removed: "9"
- note removed: "ADC RTC Shield"
- note removed: "Achtung! -------------------------------------------------- Verbindung AD4 zu LCD-Reset trennen und auf Reset des Arduino legen. AD3 zu LCD-CS ggf. trennen und auf VCC legen."
- note removed: "SCL"
- note removed: "SDA"
