File: Statemachine_ST7783_ADC/PCB/adc-rtc-shield.brd (EAGLE design)
At the start: 68.6 x 53.3 mm, 12 parts, among them IC1 RV-3029-C2, IC3 AT24C32

Commit message: -remove documentation, -add shield pcb
Parts:
- removed BATT1: 2032, El_Mech:2032_SMD
- removed C103: 100nF, rcl:C0603
- removed IC1: RV-3029-C2, crystal:SON-10
- removed IC3: AT24C32, PKJ:SOIC08
- removed JP1: (no value), pinhead:1X05/90
- removed R1: 2K2, rcl:R0603
- removed R90: 330R, rcl:R0603
- added BATT2: 2032, El_Mech:2032_SMD
- added C10, C11, C12, C13, C19, C2, C20, C21, C22, C23, C24, C25, C26, C5, C8, C9: 10n, Passiv:0805-C
- added C16, C3, C6: 100n, Passiv:0805-C
- added C27: 100nF, rcl:C0402S
- added IC2: RV_3049_C2, RTC_Quarz:5X3.2_10
- added J10, J11, J12, J13, J14, J15, J16, J9: MC1,5/2-G-3,5, PHOENIX:MC1,5/2-G-...
- added R10, R13, R14, R15, R16, R17, R6, R7, R8, R9: 2K, Passiv:R_10
- added R11, R12, R18, R19, R20, R21, R3: 10K, Passiv:R_10
- added R22: 330R, rcl:R0603
- added R4: 1K21, Passiv:R_10
- added R5: 909R, Passiv:R_10
- added U$1: TLC2543, HL_IC1:DIL_20
- R2: value 2K2 -> 10K; device rcl:R0603 -> Passiv:R_10
- moved R2 231.6 mm to (39.4, -188.5)
Connections:
- net N$29 renamed IO1
- net N$30 renamed IO0
- removed net N$12: IC1.8, R90.2
- removed net RESET: AD.5, POWER.3
- new net /CS-WDI: U$1.15
- new net 3,3V: C27.1, IC2.1
- new net AREF: IOH.8, R10.2, R13.2, R14.2, R15.2, R16.2, R17.2, R6.1, R7.1, R8.2, R9.2
- new net CLK: U$1.18
- new net DATIN: U$1.17
- new net DATOUT: U$1.16
- new net N$10: C3.2, R5.1, R6.2, U$1.13
- new net N$11: C6.2, R4.1, R7.2, U$1.14
- new net N$16: C2.2, R11.2, U$1.2
- new net N$17: C8.2, R2.2, U$1.3
- new net N$18: C9.2, R3.2, U$1.4
- new net N$19: C5.2, R12.2, U$1.1
- new net N$20: C23.2, R18.2, U$1.5
- new net N$21: C24.2, R19.2, U$1.6
- new net N$22: C25.2, R20.2, U$1.7
- new net N$23: C26.2, R21.2, U$1.8
- new net N$25: IC2.8, R22.2
- new net N$26: IC2.3
- new net N$27: BATT2.+, R22.1
- new net N$3: POWER.3
- new net SCK: IOH.6
- new net SPCK: IC2.4
- new net VCC: C16.2
- new net X1_RX4-: C13.2, J9.1, R12.1, R9.1
- new net X2_TX4-: C12.2, J10.1, R11.1, R13.1
- new net X3_RX3-: C10.2, J11.1, R10.1, R2.1
- new net X4_TX3-: C11.2, J12.1, R3.1, R8.1
- new net X5_RX2-: C19.2, J13.1, R14.1, R18.1
- new net X6_TX2-: C21.2, J14.1, R15.1, R19.1
- new net X7_RX1-: C20.2, J15.1, R16.1, R20.1
- new net X8_TX1-: C22.2, J16.1, R17.1, R21.1
- net +3V3: no longer C103.1, IC1.1, IC3.8, JP1.2, R1.2, R2.2
- net +5V: no longer JP1.1
- net AD4/SDA: now also AD.5; no longer IC1.5, IC3.5, JP1.4, R2.1
- net AD5/SCL: now also AD.6; no longer IC1.4, IC3.6, JP1.3, R1.1
- net GND: now also BATT2.-, C10.1, C11.1, C12.1, C13.1, C16.1, C19.1, C2.1, C20.1, C21.1, C22.1, C23.1, C24.1, C25.1, C26.1, C27.2, C3.1, C5.1, C6.1, C8.1, C9.1, IC2.6, J10.2, J11.2, J12.2, J13.2, J14.2, J15.2, J16.2, J9.2, R4.2, R5.2, U$1.10; no longer BATT1.-, C103.2, IC1.6, IC3.1, IC3.2, IC3.3, IC3.4, IC3.7, JP1.5
- net MISO: now also IC2.5
- net MOSI: now also IC2.9
- net N$1: now also U$1.20; no longer BATT1.+, R90.1
Routing:
- added copper zone on layer 1, net +5V
- added copper zone on layer 16, net +5V
Other:
- board text added: "Edition"
- board text added: "Limited"
- board text added: "Prototype"

Commit message: cleanup
Parts:
- renumbered U$1 to IC1
Connections:
- removed net /CS-WDI: IC1.15
- removed net 3,3V: C27.1, IC2.1
- removed net CLK: IC1.18
- removed net DATIN: IC1.17
- removed net DATOUT: IC1.16
- removed net N$1: IC1.20
- removed net N$3: POWER.3
- removed net SPCK: IC2.4
- removed net VCC: C16.2
- net +5V: now also C16.2, C27.1, IC1.20, IC2.1, R10.2, R13.2, R14.2, R15.2, R16.2, R17.2, R6.1, R7.1, R8.2, R9.2
- net AD4/SDA: now also IC1.15
- net AREF: no longer R10.2, R13.2, R14.2, R15.2, R16.2, R17.2, R6.1, R7.1, R8.2, R9.2
- net MISO: now also IC1.16
- net MOSI: now also IC1.17
- net SCK: now also IC1.18, IC2.4
Changed lines of the file:
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@@
 <attribute name="VALUE" x="26.67" y="-0.635" size="1.27" layer="27"/>
 </element>
-<element name="U$1" library="HL_IC1" package="DIL_20" value="TLC2543" x="-11.049" y="-174.625"/>
+<element name="IC1" library="HL_IC1" package="DIL_20" value="TLC2543" x="-11.049" y="-174.625"/>
 <element name="R2" library="Passiv" package="R_10" value="10K" x="39.37" y="-188.468"/>
 <element name="R3" library="Passiv" package="R_10" value="10K" x="-11.43" y="-193.421"/>
@@
 <vertex x="10.16" y="12.7"/>
 </polygon>
+<contactref element="R8" pad="2"/>
+<contactref element="R10" pad="2"/>
+<contactref element="R6" pad="1"/>
+<contactref element="R7" pad="1"/>
+<contactref element="R9" pad="2"/>
+<contactref element="R13" pad="2"/>
+<contactref element="R14" pad="2"/>
+<contactref element="R15" pad="2"/>
+<contactref element="R16" pad="2"/>
+<contactref element="R17" pad="2"/>
+<contactref element="IC2" pad="1"/>
+<contactref element="C27" pad="1"/>
+<contactref element="C16" pad="2"/>
+<contactref element="IC1" pad="20"/>
+<wire x1="-1.27" y1="-196.85" x2="-1.27" y2="-200.279" width="0" layer="19" extent="1-1"/>
+<wire x1="-3.675" y1="-189.103" x2="-1.27" y2="-196.85" width="0" layer="19" extent="1-1"/>
+<wire x1="11.049" y1="-200.279" x2="-1.27" y2="-200.279" width="0" layer="19" extent="1-1"/>
+<wire x1="11.049" y1="-196.85" x2="11.049" y2="-200.279" width="0" layer="19" extent="1-1"/>
+<wire x1="23.368" y1="-200.279" x2="11.049" y2="-200.279" width="0" layer="19" extent="1-1"/>
+<wire x1="23.368" y1="-196.85" x2="23.368" y2="-200.279" width="0" layer="19" extent="1-1"/>
+<wire x1="25.527" y1="-193.421" x2="23.368" y2="-196.85" width="0" layer="19" extent="1-1"/>
+<wire x1="35.687" y1="-200.279" x2="25.527" y2="-193.421" width="0" layer="19" extent="1-1"/>
+<wire x1="37.846" y1="-193.421" x2="35.687" y2="-200.279" width="0" layer="19" extent="1-1"/>
+<wire x1="48.006" y1="-200.279" x2="37.846" y2="-193.421" width="0" layer="19" extent="1-1"/>
+<wire x1="50.276" y1="-178.308" x2="37.846" y2="-193.421" width="0" layer="19" extent="1-1"/>
+<wire x1="35.973" y1="-171.476" x2="50.276" y2="-178.308" width="0" layer="19" extent="1-1"/>
+<wire x1="-11.049" y1="-167.005" x2="-3.675" y2="-189.103" width="0" layer="19" extent="1-1"/>
+<wire x1="38.1" y1="2.54" x2="35.973" y2="-171.476" width="0" layer="19" extent="1-1"/>
 <wire x1="30.48" y1="2.54" x2="38.1" y2="2.54" width="0" layer="19" extent="1-1"/>
 </signal>
@@
 <vertex x="0.635" y="46.355"/>
 </polygon>
-<contactref element="U$1" pad="10"/>
+<contactref element="IC1" pad="10"/>
 <contactref element="IC2" pad="6"/>
 <contactref element="C12" pad="1"/>
@@
 <contactref element="C10" pad="1"/>
 <contactref element="C2" pad="1"/>
-<contactref element="U$1" pad="10"/>
+<contactref element="IC1" pad="10"/>
 <contactref element="C3" pad="1"/>
 <contactref element="R5" pad="2"/>
@@
 <signal name="AREF" class="4">
 <contactref element="IOH" pad="8"/>
-<contactref element="R8" pad="2"/>
-<contactref element="R10" pad="2"/>
-<contactref element="R6" pad="1"/>
-<contactref element="R7" pad="1"/>
-<contactref element="R9" pad="2"/>
-<contactref element="R13" pad="2"/>
-<contactref element="R14" pad="2"/>
-<contactref element="R15" pad="2"/>
-<contactref element="R16" pad="2"/>
-<contactref element="R17" pad="2"/>
-<wire x1="-1.27" y1="-196.85" x2="-1.27" y2="-200.279" width="0" layer="19" extent="1-1"/>
-<wire x1="11.049" y1="-200.279" x2="-1.27" y2="-200.279" width="0" layer="19" extent="1-1"/>
-<wire x1="11.049" y1="-196.85" x2="11.049" y2="-200.279" width="0" layer="19" extent="1-1"/>
-<wire x1="23.368" y1="-200.279" x2="11.049" y2="-200.279" width="0" layer="19" extent="1-1"/>
-<wire x1="23.368" y1="-196.85" x2="23.368" y2="-200.279" width="0" layer="19" extent="1-1"/>
-<wire x1="25.527" y1="-193.421" x2="23.368" y2="-196.85" width="0" layer="19" extent="1-1"/>
-<wire x1="35.687" y1="-200.279" x2="25.527" y2="-193.421" width="0" layer="19" extent="1-1"/>
-<wire x1="37.846" y1="-193.421" x2="35.687" y2="-200.279" width="0" layer="19" extent="1-1"/>
-<wire x1="48.006" y1="-200.279" x2="37.846" y2="-193.421" width="0" layer="19" extent="1-1"/>
-<wire x1="23.876" y1="50.8" x2="25.527" y2="-193.421" width="0" layer="19" extent="1-1"/>
 </signal>
 <signal name="VIN" class="1">
@@
 <signal name="SCK">
 <contactref element="IOH" pad="6"/>
+<contactref element="IC2" pad="4"/>
+<contactref element="IC1" pad="18"/>
+<wire x1="38.973" y1="-171.476" x2="-5.969" y2="-167.005" width="0" layer="19" extent="1-1"/>
+<wire x1="28.956" y1="50.8" x2="-5.969" y2="-167.005" width="0" layer="19" extent="1-1"/>
 </signal>
 <signal name="+3V3">
@@
 <contactref element="IOH" pad="5"/>
 <contactref element="IC2" pad="5"/>
-<wire x1="31.496" y1="50.8" x2="39.973" y2="-171.476" width="0" layer="19" extent="1-1"/>
+<contactref element="IC1" pad="16"/>
+<wire x1="39.973" y1="-171.476" x2="-0.889" y2="-167.005" width="0" layer="19" extent="1-1"/>
+<wire x1="31.496" y1="50.8" x2="-0.889" y2="-167.005" width="0" layer="19" extent="1-1"/>
 </signal>
 <signal name="MOSI">
 <contactref element="IOH" pad="4"/>
 <contactref element="IC2" pad="9"/>
+<contactref element="IC1" pad="17"/>
+<wire x1="36.973" y1="-168.376" x2="-3.429" y2="-167.005" width="0" layer="19" extent="1-1"/>
 <wire x1="34.036" y1="50.8" x2="36.973" y2="-168.376" width="0" layer="19" extent="1-1"/>
 </signal>
@@
 <contactref element="AD" pad="5"/>
 <contactref element="IOH" pad="9"/>
-<wire x1="60.96" y1="2.54" x2="21.336" y2="50.8" width="0" layer="19" extent="1-1"/>
+<contactref element="IC1" pad="15"/>
+<wire x1="60.96" y1="2.54" x2="1.651" y2="-167.005" width="0" layer="19" extent="1-1"/>
+<wire x1="21.336" y1="50.8" x2="60.96" y2="2.54" width="0" layer="19" extent="1-1"/>
 </signal>
 <signal name="AD5/SCL">
@@
 <signal name="IO9">
 <contactref element="IOH" pad="2"/>
-</signal>
-<signal name="N$3">
-<contactref element="POWER" pad="3"/>
-</signal>
-<signal name="/CS-WDI">
-<contactref element="U$1" pad="15"/>
 </signal>
 <signal name="X2_TX4-">
@@
 <wire x1="35.814" y1="-131.064" x2="27.416" y2="-178.308" width="0" layer="19" extent="1-1"/>
 </signal>
-<signal name="CLK">
-<contactref element="U$1" pad="18"/>
-</signal>
-<signal name="DATIN">
-<contactref element="U$1" pad="17"/>
-</signal>
-<signal name="DATOUT">
-<contactref element="U$1" pad="16"/>
-</signal>
 <signal name="X8_TX1-">
 <contactref element="R17" pad="1"/>
@@
 <wire x1="2.159" y1="-163.068" x2="-0.143" y2="-184.404" width="0" layer="19" extent="1-1"/>
 </signal>
-<signal name="VCC">
-<contactref element="C16" pad="2"/>
-</signal>
-<signal name="3,3V">
-<contactref element="IC2" pad="1"/>
-<contactref element="C27" pad="1"/>
-<wire x1="35.973" y1="-171.476" x2="-3.675" y2="-189.103" width="0" layer="19" extent="1-1"/>
-</signal>
-<signal name="SPCK">
-<contactref element="IC2" pad="4"/>
-</signal>
 <signal name="N$10">
-<contactref element="U$1" pad="13"/>
+<contactref element="IC1" pad="13"/>
 <contactref element="R5" pad="1"/>
 <contactref element="R6" pad="2"/>
@@
 </signal>
 <signal name="N$11">
-<contactref element="U$1" pad="14"/>
+<contactref element="IC1" pad="14"/>
 <contactref element="R4" pad="1"/>
 <contactref element="C6" pad="2"/>
@@
 </signal>
 <signal name="N$16">
-<contactref element="U$1" pad="2"/>
+<contactref element="IC1" pad="2"/>
 <contactref element="R11" pad="2"/>
 <contactref element="C2" pad="2"/>
@@
 <contactref element="R2" pad="2"/>
 <contactref element="C8" pad="2"/>
-<contactref element="U$1" pad="3"/>
+<contactref element="IC1" pad="3"/>
 <wire x1="-5.969" y1="-174.625" x2="-9.287" y2="-189.357" width="0" layer="19" extent="1-1"/>
 <wire x1="49.53" y1="-188.468" x2="-5.969" y2="-174.625" width="0" layer="19" extent="1-1"/>
@@
 <contactref element="R3" pad="2"/>
 <contactref element="C9" pad="2"/>
-<contactref element="U$1" pad="4"/>
+<contactref element="IC1" pad="4"/>
 <wire x1="-5.35" y1="-189.357" x2="-1.27" y2="-193.421" width="0" layer="19" extent="1-1"/>
 <wire x1="-3.429" y1="-174.625" x2="-5.35" y2="-189.357" width="0" layer="19" extent="1-1"/>
@@
 <contactref element="R12" pad="2"/>
 <contactref element="C5" pad="2"/>
-<contactref element="U$1" pad="1"/>
+<contactref element="IC1" pad="1"/>
 <wire x1="44.307" y1="-184.404" x2="-11.049" y2="-174.625" width="0" layer="19" extent="1-1"/>
 <wire x1="48.006" y1="-196.85" x2="44.307" y2="-184.404" width="0" layer="19" extent="1-1"/>
@@
 <signal name="N$20">
 <contactref element="R18" pad="2"/>
-<contactref element="U$1" pad="5"/>
+<contactref element="IC1" pad="5"/>
 <contactref element="C23" pad="2"/>
 <wire x1="18.145" y1="-184.404" x2="-1.27" y2="-203.708" width="0" layer="19" extent="1-1"/>
@@
 </signal>
 <signal name="N$21">
-<contactref element="U$1" pad="6"/>
+<contactref element="IC1" pad="6"/>
 <contactref element="R19" pad="2"/>
 <contactref element="C24" pad="2"/>
@@
 </signal>
 <signal name="N$22">
-<contactref element="U$1" pad="7"/>
+<contactref element="IC1" pad="7"/>
 <contactref element="R20" pad="2"/>
 <contactref element="C25" pad="2"/>
@@
 </signal>
 <signal name="N$23">
-<contactref element="U$1" pad="8"/>
+<contactref element="IC1" pad="8"/>
 <contactref element="R21" pad="2"/>
 <contactref element="C26" pad="2"/>
@@
 <wire x1="-2.159" y1="-149.27" x2="3.214" y2="-189.103" width="0" layer="19" extent="1-1"/>
 </signal>
-<signal name="N$1">
-<contactref element="U$1" pad="20"/>
-</signal>
 </signals>

Commit message: edit board.
Parts:
- removed J10, J11, J12, J13, J14, J15, J16, J9: MC1,5/2-G-3,5, PHOENIX:MC1,5/2-G-...
- added JP1: 9x1F-H8.5, pinhead:1X09/90
- added JP2, JP3, JP4, JP5, JP6, JP7: (no value), pinhead:1X01
- C27: device rcl:C0402S -> rcl:C0603
- R10, R13, R14, R15, R16, R17, R4, R5, R6, R8, R9: device Passiv:R_10 -> resistor:0207/10
- R11, R12, R18, R19, R2, R20, R21, R3, R7: device Passiv:R_10 -> resistor:0207/12
- R22: device rcl:R0603 -> rcl:0207/10
- moved R13 238.1 mm to (10.2, 36.8), turned to 90 degrees
- moved R9 236.3 mm to (7.62, 39.4), turned to 90 degrees
- moved R22 234.7 mm to (45.7, 41.9), turned to 180 degrees
- moved C27 231.6 mm to (31.4, 39.9), flipped to the bottom
- moved R12 231.5 mm to (24.1, 34.3)
- moved R10 231.1 mm to (12.7, 34.3), turned to 90 degrees
- moved R18 230.6 mm to (24.1, 24.1)
- moved R8 230.2 mm to (15.2, 31.8), turned to 90 degrees
- moved R11 228.6 mm to (24.1, 31.8)
- moved R19 226.5 mm to (24.1, 21.6)
- moved R4 224.4 mm to (44.5, 26.7), turned to 90 degrees
- moved R20 223.0 mm to (24.1, 19.1)
- moved R3 222.9 mm to (24.1, 26.7)
- moved C8 221.7 mm to (26.7, 29.2), flipped to the bottom, turned to 180 degrees
- moved R21 220.2 mm to (24.1, 16.5)
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Connections:
- removed net N$26: IC2.3
- removed net N$27: BATT2.+, R22.1
- new net +BAT: BATT2.+, JP4.1, JP5.1, R22.1
- new net AD4/SDA': AD.5
- new net AD5/SCL': AD.6
- net +5V: now also JP6.1, JP7.1; no longer POWER.2
- net AD4/SDA: now also IC2.3; no longer AD.5, IC1.15
- net AD5/SCL: now also IC1.15; no longer AD.6
- net GND: now also JP1.1, JP2.1, JP3.1; no longer J10.2, J11.2, J12.2, J13.2, J14.2, J15.2, J16.2, J9.2
- net X1_RX4-: now also JP1.9; no longer J9.1
- net X2_TX4-: now also JP1.8; no longer J10.1
- net X3_RX3-: now also JP1.7; no longer J11.1
- net X4_TX3-: now also JP1.6; no longer J12.1
- net X5_RX2-: now also JP1.5; no longer J13.1
- net X6_TX2-: now also JP1.4; no longer J14.1
- net X7_RX1-: now also JP1.3; no longer J15.1
- net X8_TX1-: now also JP1.2; no longer J16.1
Routing:
- net +5V: track 0.00 -> 181.3 mm
- net AD5/SCL: track 0.00 -> 48.7 mm
- net SCK: track 0.00 -> 45.9 mm
- net MOSI: track 0.00 -> 39.0 mm
- net MISO: track 0.00 -> 33.8 mm
- net AD4/SDA: track 0.00 -> 21.3 mm
- net N$10: track 0.00 -> 17.8 mm
- net X8_TX1-: track 0.00 -> 16.1 mm
- net X7_RX1-: track 0.00 -> 16.1 mm
- net X6_TX2-: track 0.00 -> 16.1 mm
- net X5_RX2-: track 0.00 -> 16.1 mm
- net X4_TX3-: track 0.00 -> 16.1 mm
- net X3_RX3-: track 0.00 -> 16.1 mm
- net X2_TX4-: track 0.00 -> 16.1 mm
- net X1_RX4-: track 0.00 -> 16.1 mm
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- removed copper zone on layer 1, net +5V
- removed copper zone on layer 16, net +5V
- removed copper zone on layer 1, net GND
Other:
- board text added: "TINO 1.0"
- board text removed: "Edition"
- board text removed: "Limited"
- board text removed: "Prototype"

Commit message: Remove Arduino text.
Other:
- board text removed: "#"
- board text removed: "0"
- board text removed: "10"
- board text removed: "11"
- board text removed: "12"
- board text removed: "13"
- board text removed: "2"
- board text removed: "3"
- board text removed: "3V3"
- board text removed: "4"
- board text removed: "5"
- board text removed: "5V"
- board text removed: "6"
- board text removed: "7"
- board text removed: "8"
- board text removed: "9"
- board text removed: "A0"
- board text removed: "A1"
- board text removed: "A2"
- board text removed: "A3"
- board text removed: "A4"
- board text removed: "A5"
- board text removed: "ANALOG IN"
- board text removed: "AREF"
- board text removed: "ATMEGA328"
- board text removed: "Arduino"
- board text removed: "D.Cuartielles"
- board text removed: "D.Mellis"
- board text removed: "DIGITAL"
- board text removed: "G.Martino"
- board text removed: "GND"
- board text removed: "IOREF"
- board text removed: "ITALY"
- board text removed: "L"
- board text removed: "M.Banzi"
- board text removed: "MADE IN"
- board text removed: "ON"
- board text removed: "PC1"
- board text removed: "PC2"
- board text removed: "RESET"
- board text removed: "T.Igoe"
- board text removed: "TM"
- board text removed: "UNO"
- board text removed: "VIN"
- board text removed: "[#=PWM]"
- board text removed: "designed by"
- board text removed: "tinker it"
- board text removed: "www.arduino.cc"
