File: Statemachine_ST7783_ADC/PCB/adc-rtc-shield.brd (EAGLE design)
At the start: 68.6 x 53.3 mm, 55 parts, among them IC1 TLC2543, IC2 RV_3049_C2

Commit message: Voltage devider changed.
Parts:
- R4: value 1K21 -> 1K5
Changed lines of the file:
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@@
 <element name="R2" library="resistor" package="0207/12" value="10K" x="24.13" y="29.21"/>
 <element name="R3" library="resistor" package="0207/12" value="10K" x="24.13" y="26.67"/>
-<element name="R4" library="resistor" package="0207/10" value="1K21" x="44.45" y="26.67" rot="R90"/>
+<element name="R4" library="resistor" package="0207/10" value="1K5" x="44.45" y="26.67" rot="R90"/>
 <element name="R5" library="resistor" package="0207/10" value="909R" x="24.13" y="13.97" rot="R180"/>
 <element name="R6" library="resistor" package="0207/10" value="2K" x="24.13" y="11.43"/>
