File: MiniTino/PCB/adc-rtc-shield.brd (EAGLE design)
At the start: 68.6 x 53.3 mm, 51 parts, among them IC1 TLC2543, IC2 RV_3049_C2

Commit message: Brd.
Routing:
- net N$18: track 25.2 -> 0.00 mm
- net N$20: track 21.0 -> 0.00 mm
- net N$21: track 18.2 -> 0.00 mm
- net N$22: track 16.9 -> 0.00 mm
- net N$23: track 16.4 -> 0.00 mm
Changed lines of the file:
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@@
 <grid distance="0.05" unitdist="inch" unit="inch" style="lines" multiple="1" display="no" altdistance="0.025" altunitdist="inch" altunit="inch"/>
 <layers>
-<layer number="1" name="Top" color="4" fill="1" visible="yes" active="yes"/>
+<layer number="1" name="Top" color="4" fill="1" visible="no" active="yes"/>
 <layer number="16" name="Bottom" color="1" fill="1" visible="yes" active="yes"/>
 <layer number="17" name="Pads" color="2" fill="1" visible="yes" active="yes"/>
@@
 <layer number="19" name="Unrouted" color="6" fill="1" visible="yes" active="yes"/>
 <layer number="20" name="Dimension" color="15" fill="1" visible="yes" active="yes"/>
-<layer number="21" name="tPlace" color="7" fill="1" visible="yes" active="yes"/>
+<layer number="21" name="tPlace" color="7" fill="1" visible="no" active="yes"/>
 <layer number="22" name="bPlace" color="7" fill="1" visible="no" active="yes"/>
-<layer number="23" name="tOrigins" color="15" fill="1" visible="yes" active="yes"/>
+<layer number="23" name="tOrigins" color="15" fill="1" visible="no" active="yes"/>
 <layer number="24" name="bOrigins" color="15" fill="1" visible="yes" active="yes"/>
 <layer number="25" name="tNames" color="7" fill="1" visible="no" active="yes"/>
@@
 <contactref element="JP1" pad="16"/>
 <contactref element="JP2" pad="3"/>
+<wire x1="51.07" y1="10.795" x2="55.88" y2="29.21" width="0" layer="19" extent="1-1"/>
 <wire x1="42.76" y1="10.795" x2="51.07" y2="10.795" width="0" layer="19" extent="1-1"/>
 <wire x1="42.91" y1="6.985" x2="42.76" y2="10.795" width="0" layer="19" extent="1-1"/>
 <wire x1="43.18" y1="2.54" x2="42.91" y2="6.985" width="0" layer="19" extent="1-1"/>
-<wire x1="13.86979375" y1="40.7469375" x2="16.51" y2="41.64" width="0" layer="19" extent="1-16"/>
-<wire x1="19.33" y1="39.91" x2="16.51" y2="41.64" width="0" layer="19" extent="1-16"/>
+<wire x1="40.64" y1="2.54" x2="43.18" y2="2.54" width="0" layer="19" extent="1-1"/>
 <wire x1="37.68" y1="10.795" x2="42.76" y2="10.795" width="0" layer="19" extent="1-1"/>
 <wire x1="35.83" y1="6.985" x2="37.68" y2="10.795" width="0" layer="19" extent="1-1"/>
+<wire x1="30.48" y1="21.59" x2="37.68" y2="10.795" width="0" layer="19" extent="1-1"/>
+<wire x1="24.13" y1="20.59" x2="30.48" y2="21.59" width="0" layer="19" extent="16-16"/>
+<wire x1="24.13" y1="24.4" x2="24.13" y2="20.59" width="0" layer="19" extent="16-16"/>
+<wire x1="24.13" y1="28.21" x2="24.13" y2="24.4" width="0" layer="19" extent="16-16"/>
+<wire x1="24.13" y1="32.02" x2="24.13" y2="28.21" width="0" layer="19" extent="16-16"/>
+<wire x1="24.13" y1="16.78" x2="24.13" y2="20.59" width="0" layer="19" extent="16-16"/>
+<wire x1="24.13" y1="12.97" x2="24.13" y2="16.78" width="0" layer="19" extent="16-16"/>
+<wire x1="24.13" y1="37.83" x2="24.13" y2="32.02" width="0" layer="19" extent="16-16"/>
+<wire x1="24.13" y1="39.64" x2="24.13" y2="37.83" width="0" layer="19" extent="16-16"/>
+<wire x1="19.33" y1="39.91" x2="24.13" y2="39.64" width="0" layer="19" extent="1-16"/>
+<wire x1="16.51" y1="41.64" x2="19.33" y2="39.91" width="0" layer="19" extent="1-16"/>
+<wire x1="13.86979375" y1="40.7469375" x2="16.51" y2="41.64" width="0" layer="19" extent="1-16"/>
+<wire x1="16.51" y1="37.83" x2="19.33" y2="39.91" width="0" layer="19" extent="1-16"/>
+<wire x1="16.51" y1="34.02" x2="16.51" y2="37.83" width="0" layer="19" extent="16-16"/>
+<wire x1="16.51" y1="30.21" x2="16.51" y2="34.02" width="0" layer="19" extent="16-16"/>
+<wire x1="16.51" y1="26.4" x2="16.51" y2="30.21" width="0" layer="19" extent="16-16"/>
+<wire x1="16.51" y1="22.59" x2="16.51" y2="26.4" width="0" layer="19" extent="16-16"/>
+<wire x1="16.51" y1="18.78" x2="16.51" y2="22.59" width="0" layer="19" extent="16-16"/>
+<wire x1="16.51" y1="14.97" x2="16.51" y2="18.78" width="0" layer="19" extent="16-16"/>
+<wire x1="5.08" y1="41.91" x2="13.86979375" y2="40.7469375" width="0" layer="19" extent="1-1"/>
+<wire x1="5.08" y1="44.45" x2="5.08" y2="41.91" width="0" layer="19" extent="1-1"/>
+<wire x1="5.08" y1="46.99" x2="5.08" y2="44.45" width="0" layer="19" extent="1-1"/>
+<wire x1="5.08" y1="39.37" x2="5.08" y2="41.91" width="0" layer="19" extent="1-1"/>
+<wire x1="5.08" y1="36.83" x2="5.08" y2="39.37" width="0" layer="19" extent="1-1"/>
+<wire x1="5.08" y1="34.29" x2="5.08" y2="36.83" width="0" layer="19" extent="1-1"/>
+<wire x1="5.08" y1="31.75" x2="5.08" y2="34.29" width="0" layer="19" extent="1-1"/>
+<wire x1="5.08" y1="29.21" x2="5.08" y2="31.75" width="0" layer="19" extent="1-1"/>
 <wire x1="17.78" y1="5.416" x2="16.51" y2="14.97" width="0" layer="19" extent="1-16"/>
+<wire x1="26.416" y1="50.8" x2="24.13" y2="39.64" width="0" layer="19" extent="16-16"/>
+<wire x1="5.08" y1="11.43" x2="16.51" y2="14.97" width="0" layer="19" extent="16-16"/>
 </signal>
 <signal name="AREF" class="4">
@@
 <contactref element="C9" pad="2"/>
 <contactref element="IC1" pad="4"/>
+<wire x1="24.13" y1="30.21" x2="45.72" y2="21.59" width="0" layer="19" extent="16-16"/>
 <wire x1="19.05" y1="30.06" x2="24.13" y2="30.21" width="0" layer="19" extent="16-16"/>
-<wire x1="24.13" y1="30.21" x2="25.67" y2="30.21" width="0.4064" layer="1"/>
-<wire x1="25.67" y1="30.21" x2="29.21" y2="26.67" width="0.4064" layer="1"/>
-<wire x1="29.21" y1="26.67" x2="40.64" y2="26.67" width="0.4064" layer="1"/>
-<wire x1="40.64" y1="26.67" x2="45.72" y2="21.59" width="0.4064" layer="1"/>
 </signal>
 <signal name="N$19">
@@
 <contactref element="IC1" pad="5"/>
 <contactref element="C23" pad="2"/>
+<wire x1="24.13" y1="26.4" x2="43.18" y2="21.59" width="0" layer="19" extent="16-16"/>
 <wire x1="19.05" y1="26.25" x2="24.13" y2="26.4" width="0" layer="19" extent="16-16"/>
-<wire x1="24.13" y1="26.4" x2="26.94" y2="26.4" width="0.4064" layer="1"/>
-<wire x1="26.94" y1="26.4" x2="27.94" y2="25.4" width="0.4064" layer="1"/>
-<wire x1="27.94" y1="25.4" x2="39.37" y2="25.4" width="0.4064" layer="1"/>
-<wire x1="39.37" y1="25.4" x2="43.18" y2="21.59" width="0.4064" layer="1"/>
 </signal>
 <signal name="N$21">
@@
 <contactref element="R19" pad="2"/>
 <contactref element="C24" pad="2"/>
+<wire x1="24.13" y1="22.59" x2="40.64" y2="21.59" width="0" layer="19" extent="16-16"/>
 <wire x1="19.05" y1="22.44" x2="24.13" y2="22.59" width="0" layer="19" extent="16-16"/>
-<wire x1="24.13" y1="22.59" x2="26.4" y2="22.59" width="0.4064" layer="1"/>
-<wire x1="26.4" y1="22.59" x2="27.94" y2="24.13" width="0.4064" layer="1"/>
-<wire x1="27.94" y1="24.13" x2="38.1" y2="24.13" width="0.4064" layer="1"/>
-<wire x1="38.1" y1="24.13" x2="40.64" y2="21.59" width="0.4064" layer="1"/>
 </signal>
 <signal name="N$22">
@@
 <contactref element="R20" pad="2"/>
 <contactref element="C25" pad="2"/>
+<wire x1="24.13" y1="18.78" x2="38.1" y2="21.59" width="0" layer="19" extent="16-16"/>
 <wire x1="19.05" y1="18.63" x2="24.13" y2="18.78" width="0" layer="19" extent="16-16"/>
-<wire x1="24.13" y1="18.78" x2="26.4" y2="18.78" width="0.4064" layer="1"/>
-<wire x1="26.4" y1="18.78" x2="27.94" y2="20.32" width="0.4064" layer="1"/>
-<wire x1="27.94" y1="20.32" x2="27.94" y2="21.59" width="0.4064" layer="1"/>
-<wire x1="27.94" y1="21.59" x2="29.21" y2="22.86" width="0.4064" layer="1"/>
-<wire x1="29.21" y1="22.86" x2="36.83" y2="22.86" width="0.4064" layer="1"/>
-<wire x1="36.83" y1="22.86" x2="38.1" y2="21.59" width="0.4064" layer="1"/>
 </signal>
 <signal name="N$23">
@@
 <contactref element="R21" pad="2"/>
 <contactref element="C26" pad="2"/>
+<wire x1="24.13" y1="14.97" x2="35.56" y2="21.59" width="0" layer="19" extent="16-16"/>
 <wire x1="19.05" y1="14.82" x2="24.13" y2="14.97" width="0" layer="19" extent="16-16"/>
-<wire x1="24.13" y1="14.97" x2="27.67" y2="14.97" width="0.4064" layer="16"/>
-<wire x1="27.67" y1="14.97" x2="29.21" y2="16.51" width="0.4064" layer="16"/>
-<wire x1="29.21" y1="16.51" x2="34.29" y2="16.51" width="0.4064" layer="16"/>
-<wire x1="34.29" y1="16.51" x2="35.56" y2="17.78" width="0.4064" layer="16"/>
-<wire x1="35.56" y1="17.78" x2="35.56" y2="21.59" width="0.4064" layer="16"/>
 </signal>
 <signal name="N$25">
